File: gfmpw1_breakout.kicad_sch (KiCad schematic)
At the start: 19 parts, among them J1 Conn_01x20_Pin, J2 Conn_01x20_Pin, U1 AMS1117-3.3, U1 Caravel, U1 SN74LV1T34DCK, U3 MCP1319MT-29LE-OT, U5 W25Q32FVSS

Commit message: Revision 2
Parts:
- removed R1, R3: 1K, Resistor_SMD:R_1206_3216Metric_Pad1.30x1.75mm_HandSolder, symbol Device:R
- removed R2: 10K, Resistor_SMD:R_1206_3216Metric_Pad1.30x1.75mm_HandSolder, symbol Device:R
- removed U1 (x4): SN74LV1T34DCK, Package_TO_SOT_SMD:SOT-23-5, symbol Logic_LevelTranslator:SN74LV1T34DCK
- added J3: Conn_01x05, Connector_PinHeader_2.54mm:PinHeader_1x05_P2.54mm_Vertical, symbol Connector_Generic:Conn_01x05
- added R5, R6: 1K, Resistor_SMD:R_1206_3216Metric_Pad1.30x1.75mm_HandSolder, symbol Device:R
- added U5, U6, U7, U8: SN74LV1T126DCK, Package_TO_SOT_SMD:SOT-23-5, symbol TholinsStuff:SN74LV1T126DCK
- C1, C2: value 100nF -> 1µF; footprint Capacitor_SMD:C_1206_3216Metric_Pad1.33x1.80mm_HandSolder -> Capacitor_SMD:C_0805_2012Metric_Pad1.18x1.45mm_HandSolder
- C3: value 0.1µF -> 1µF; footprint Capacitor_SMD:C_1206_3216Metric_Pad1.33x1.80mm_HandSolder -> Capacitor_SMD:C_0805_2012Metric_Pad1.18x1.45mm_HandSolder
- U2: renamed from U5; footprint Package_DIP:DIP-8_W7.62mm -> Package_SO:SOIC-8_5.3x5.3mm_P1.27mm
- renumbered U1 to U4
Connections:
- net +3V3: now also U2.3 (~{WP}(D2)), U2.7 (~{HOLD}(D3)), U5.5 (VCC), U7.5 (VCC), U8.5 (VCC)
- net +5V: now also R5.2, R6.2, U6.5 (VCC)
- net FLASH_CLK: now also J3.5 (Pin_5), U8.4 (Y)
- net FLASH_CSB: now also J3.4 (Pin_4), U5.4 (Y)
- net FLASH_SDI: now also J3.3 (Pin_3), U7.4 (Y)
- net FLASH_SDO: now also J3.2 (Pin_2), U6.2 (A)
- net GND: now also U5.3 (GND), U6.3 (GND), U7.3 (GND), U8.3 (GND)
- net at U4.26 (flash_io0): now also U7.2 (A)
- net at U4.24 (flash_csb): now also U5.2 (A)
- net at U4.25 (flash_clk): now also U8.2 (A)
- net at U4.27 (flash_io1): now also U6.4 (Y)
- net at U4.34 (mprj_io[3]_CSB): now also R5.1
- net ~{PGM}: now reaches U3.4 (~{MR})
- net ~{PGM}: now also J3.1 (Pin_1), R6.1, U5.1 (OE), U6.1 (OE), U7.1 (OE), U8.1 (OE)
- no-connect marks 2 -> 1
