File: gfmpw1_breakout.kicad_pcb (KiCad board)
At the start: 4 copper layers, 20.3 x 53.3 mm, 19 parts, among them J1 Conn_01x20_Pin, J2 Conn_01x20_Pin, U1 AMS1117-3.3, U2 W25Q32FVSS, U3 MCP1319MT-29LE-OT, U4 Caravel, U5 SN74LV1T34DCK, U6 SN74LV1T34DCK, U7 SN74LV1T34DCK, U8 SN74LV1T34DCK

Commit message: Revision 2
Parts:
- removed R1, R3: 1K, Resistor_SMD:R_1206_3216Metric_Pad1.30x1.75mm_HandSolder
- removed R2: 10K, Resistor_SMD:R_1206_3216Metric_Pad1.30x1.75mm_HandSolder
- added J3: Conn_01x05, Connector_PinHeader_2.54mm:PinHeader_1x05_P2.54mm_Vertical, F.Cu at (123.7, 70.8)
- added R5: 1K, Resistor_SMD:R_1206_3216Metric_Pad1.30x1.75mm_HandSolder, F.Cu at (131.0, 113.0)
- added R6: 1K, Resistor_SMD:R_1206_3216Metric_Pad1.30x1.75mm_HandSolder, F.Cu at (128.0, 79.8)
- C1, C2: value 100nF -> 1µF; footprint Capacitor_SMD:C_1206_3216Metric_Pad1.33x1.80mm_HandSolder -> Capacitor_SMD:C_0805_2012Metric_Pad1.18x1.45mm_HandSolder
- C3: value 0.1µF -> 1µF; footprint Capacitor_SMD:C_1206_3216Metric_Pad1.33x1.80mm_HandSolder -> Capacitor_SMD:C_0805_2012Metric_Pad1.18x1.45mm_HandSolder
- U2: footprint Package_DIP:DIP-8_W7.62mm -> Package_SO:SOIC-8_5.3x5.3mm_P1.27mm
- U5, U6, U7, U8: value SN74LV1T34DCK -> SN74LV1T126DCK
- moved U2 4.88 mm to (128.2, 75.5)
- moved U5 0.20 mm to (131.5, 93.2)
- moved U8 0.12 mm to (131.2, 97.5)
- moved U7 0.11 mm to (126.0, 97.5)
Connections:
- U2 pad 3: Net-(U2-~{WP}(D2)) -> +3V3
- U2 pad 7: Net-(U2-~{HOLD}(D3)) -> +3V3
- U3 pad 4: Net-(U3-~{MR}) -> ~{PGM}
- U4 pad 34: unconnected-(U4-mprj_io[3]_CSB-Pad34) -> Net-(U4-mprj_io[3]_CSB)
- U5 pad 1: unconnected-(U5-NC-Pad1) -> ~{PGM}
- U6 pad 1: unconnected-(U6-NC-Pad1) -> ~{PGM}
- U7 pad 1: unconnected-(U7-NC-Pad1) -> ~{PGM}
- U8 pad 1: unconnected-(U8-NC-Pad1) -> ~{PGM}
Routing:
- net ~{PGM}: track 0.00 -> 74.0 mm, vias 0 -> 3
- net FLASH_SDI: track 21.5 -> 36.6 mm, vias 1 -> 3
- net +5V: track 79.1 -> 92.2 mm
- net GND: track 65.5 -> 76.5 mm, vias 10 -> 11
- net FLASH_CLK: track 22.5 -> 30.6 mm, vias 1 -> 3
- net FLASH_CSB: track 25.4 -> 33.0 mm, vias 1 -> 4
- net Net-(U2-~{WP}(D2)): track 6.31 -> 0.00 mm
- net FLASH_SDO: track 20.3 -> 26.5 mm, vias 0 -> 2
- net +3V3: track 55.4 -> 61.5 mm
- net Net-(U4-mprj_io[3]_CSB): track 0.00 -> 5.59 mm, vias 0 -> 2
- net Net-(U2-~{HOLD}(D3)): track 3.02 -> 0.00 mm
- net Net-(U3-~{MR}): track 2.39 -> 0.00 mm
Other:
- board text added: "0110"
- board text removed: "0079"

Commit message: Documentation updates & minor PCB file fix.
Parts:
- moved J3 10.2 mm to (133.8, 71.0), turned to -90 degrees
Routing:
- net ~{PGM}: track 74.0 -> 85.2 mm
- net FLASH_CLK: track 30.6 -> 38.0 mm
- net FLASH_SDO: track 26.5 -> 33.0 mm, vias 2 -> 3
- net FLASH_CSB: track 33.0 -> 29.9 mm
- net FLASH_SDI: track 36.6 -> 35.5 mm
